File: pcb/Rev 1.brd (EAGLE design)
At the start: 76.8 x 76.8 mm, 216 parts, among them J1 3220-10-0100-00, J2 10118194-0001LF, J3 B2B-PH-K-S(LF)(SN), Q1 MMBT3904,215MMBT3904,215, Q12 MMBT3904,215MMBT3904,215, Q13 MMBT3904,215MMBT3904,215, Q14 MMBT3904,215MMBT3904,215, Q15 MMBT3904,215MMBT3904,215, Q16 TEFT4300, Q17 TEFT4300, Q18 TEFT4300, Q19 TEFT4300, Q20 MMBT3904,215MMBT3904,215, Q21 MMBT3904,215MMBT3904,215, Q22 MMBT3904,215MMBT3904,215, Q23 MMBT3904,215MMBT3904,215, Q24 TEFT4300, Q25 TEFT4300, Q26 TEFT4300, Q27 TEFT4300, Q28 SI7157DP, Q29 SI7157DP, Q30 MMBT3906, Q31 MMBT3906, Q32 SI7157DP, Q33 MMBT3906, Q34 MMBT3906, U1 ATSAMD21G18A-MU, U10 DRV8871, U11 PCAL6416A, U12 MAX7315, U2 AP3441, U3 TPS61089, U4 BNO055, U5 MCP73811, U7 DRV8871, U8 DRV8871, U9 DRV8871

Commit message: Created ground plane and fixed DRC
Routing:
- net GND: track 0.00 -> 36.1 mm, vias 0 -> 65
- net +3V7: track 150.4 -> 145.8 mm
- net +3V3: track 500.6 -> 499.9 mm
- added copper zone on layer 1, net GND
- added copper zone on layer 16, net GND
