File: pcb/EncoderR1.sch (EAGLE design)
At the start: 8 parts, among them U1 TLE49462KHTSA1, U2 TLE49462KHTSA1

Commit message: Created encoder board
Parts:
- C1, C2: device Micromouse 2020:CAPACITOR0805 -> Micromouse 2020:CAPACITOR0603
- R1, R2: device Micromouse 2020:RESISTOR0805 -> Micromouse 2020:RESISTOR0603
Connections:
- removed net N$1: R1.P$1, U1.Q
- removed net N$2: R2.P$1, U2.Q
- net OUTA: now also R2.P$1, U2.Q
- net OUTB: now also R1.P$1, U1.Q
Changed lines of the file:
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@@
 <?xml version="1.0" encoding="utf-8"?>
 <!DOCTYPE eagle SYSTEM "eagle.dtd">
-<eagle version="9.2.2">
+<eagle version="9.5.2">
 <drawing>
 <settings>
@@
 <part name="P+1" library="Micromouse 2020" deviceset="+3V3" device=""/>
 <part name="GND1" library="Micromouse 2020" deviceset="GND" device=""/>
-<part name="C1" library="Micromouse 2020" deviceset="CAPACITOR" device="0805" value="0.1uF"/>
+<part name="C1" library="Micromouse 2020" deviceset="CAPACITOR" device="0603" package3d_urn="urn:adsk.eagle:package:16053670/1" value="0.1uF"/>
 <part name="L1" library="Micromouse 2020" deviceset="MOTOR" device=""/>
-<part name="C2" library="Micromouse 2020" deviceset="CAPACITOR" device="0805" value="3.3nF"/>
+<part name="C2" library="Micromouse 2020" deviceset="CAPACITOR" device="0603" package3d_urn="urn:adsk.eagle:package:16053670/1" value="3.3nF"/>
 <part name="U1" library="Micromouse 2020" deviceset="TLE49462KHTSA1" device="" package3d_urn="urn:adsk.eagle:package:14494850/1"/>
-<part name="R1" library="Micromouse 2020" deviceset="RESISTOR" device="0805" value="10k"/>
+<part name="R1" library="Micromouse 2020" deviceset="RESISTOR" device="0603" package3d_urn="urn:adsk.eagle:package:16053670/1" value="10k"/>
 <part name="P+2" library="Micromouse 2020" deviceset="+3V3" device=""/>
 <part name="GND2" library="Micromouse 2020" deviceset="GND" device=""/>
 <part name="U2" library="Micromouse 2020" deviceset="TLE49462KHTSA1" device="" package3d_urn="urn:adsk.eagle:package:14494850/1"/>
-<part name="R2" library="Micromouse 2020" deviceset="RESISTOR" device="0805" value="10k"/>
+<part name="R2" library="Micromouse 2020" deviceset="RESISTOR" device="0603" package3d_urn="urn:adsk.eagle:package:16053670/1" value="10k"/>
 <part name="P+3" library="Micromouse 2020" deviceset="+3V3" device=""/>
 <part name="GND3" library="Micromouse 2020" deviceset="GND" device=""/>
@@
 <label x="7.62" y="0" size="1.778" layer="95"/>
 </segment>
+<segment>
+<pinref part="U1" gate="G$1" pin="Q"/>
+<wire x1="45.72" y1="2.54" x2="48.26" y2="2.54" width="0.1524" layer="91"/>
+<pinref part="R1" gate="G$1" pin="P$1"/>
+<wire x1="48.26" y1="2.54" x2="48.26" y2="5.08" width="0.1524" layer="91"/>
+<label x="45.72" y="2.54" size="1.778" layer="95"/>
+</segment>
 </net>
 <net name="OUTA" class="0">
@@
 <wire x1="5.08" y1="2.54" x2="15.24" y2="2.54" width="0.1524" layer="91"/>
 <label x="7.62" y="2.54" size="1.778" layer="95"/>
+</segment>
+<segment>
+<pinref part="U2" gate="G$1" pin="Q"/>
+<wire x1="63.5" y1="2.54" x2="66.04" y2="2.54" width="0.1524" layer="91"/>
+<pinref part="R2" gate="G$1" pin="P$1"/>
+<wire x1="66.04" y1="2.54" x2="66.04" y2="5.08" width="0.1524" layer="91"/>
+<label x="63.5" y="2.54" size="1.778" layer="95"/>
 </segment>
 </net>
@@
 </segment>
 </net>
-<net name="N$1" class="0">
-<segment>
-<pinref part="U1" gate="G$1" pin="Q"/>
-<wire x1="45.72" y1="2.54" x2="48.26" y2="2.54" width="0.1524" layer="91"/>
-<pinref part="R1" gate="G$1" pin="P$1"/>
-<wire x1="48.26" y1="2.54" x2="48.26" y2="5.08" width="0.1524" layer="91"/>
-</segment>
-</net>
-<net name="N$2" class="0">
-<segment>
-<pinref part="U2" gate="G$1" pin="Q"/>
-<wire x1="63.5" y1="2.54" x2="66.04" y2="2.54" width="0.1524" layer="91"/>
-<pinref part="R2" gate="G$1" pin="P$1"/>
-<wire x1="66.04" y1="2.54" x2="66.04" y2="5.08" width="0.1524" layer="91"/>
-</segment>
-</net>
